File: Prinsip/Prinsip.sch (KiCad schematic (older format))
At the start: 46 parts

Commit message: upd
Parts:
- gave numbers to parts that had none: 1
Connections:
- new net: DD40.~ (~LD), DD41.~ (Uоп) (x8)
Changed lines of the file:
@@
 $EndComp
 $Comp
-L Switch:SW_DIP_x08 SW?
+L Switch:SW_DIP_x08 SW1
 U 1 1 6169F626
 P 1450 5200
-F 0 "SW?" H 1450 5867 50  0000 C CNN
+F 0 "SW1" H 1450 5867 50  0000 C CNN
 F 1 "SW_DIP_x08" H 1450 5776 50  0000 C CNN
 F 2 "" H 1450 5200 50  0001 C CNN
