File: Prinsip/Prinsip.sch (KiCad schematic (older format))
At the start: 46 parts, among them SW1 SW_DIP_x08

Commit message: Added caps
Parts:
- added C1, C2...C4: con-Prinsip, symbol rescue:con-Prinsip
- DD39: symbol Prinsip:COUNTER -> Prinsip-rescue:COUNTER-Prinsip
- R1, R2: symbol Принципиально-rescue:R_Small-Device -> Prinsip-rescue:R_Small-Device-Принципиально-rescue
- SW1: symbol Switch:SW_DIP_x08 -> Prinsip-rescue:SW_DIP_x08-Switch
- U?: symbol Принципиально-rescue:TAB-Prinsip -> Prinsip-rescue:TAB-Prinsip-Принципиально-rescue
- ZQ1: symbol Принципиально-rescue:Resonator-Device -> Prinsip-rescue:Resonator-Device-Принципиально-rescue
Connections:
- new net: DD40.~ (~LD), DD41.~ (Uоп) (x8)
- new net: C1.~, C2...C4.~ (x2)
Other:
- note added: "+"
Changed lines of the file:
@@
 $EndComp
 $Comp
-L power:+24V #PWR?
+L Prinsip-rescue:+24V-power #PWR?
 U 1 1 6168DD81
 P 15050 5750
@@
 $EndComp
 $Comp
-L Switch:SW_DIP_x08 SW1
+L Prinsip-rescue:SW_DIP_x08-Switch SW1
 U 1 1 6169F626
 P 1450 5200
@@
 	1050 5400 1050 5300
 $Comp
-L power:+5V #PWR?
+L Prinsip-rescue:+5V-power #PWR?
 U 1 1 616F5484
 P 1050 4650
@@
 CLK
 $Comp
-L Prinsip:COUNTER DD39
+L Prinsip-rescue:COUNTER-Prinsip DD39
 U 1 1 618F24BD
 P 12850 4800
@@
 $EndComp
 $Comp
-L Принципиально-rescue:Resonator-Device ZQ1
+L Prinsip-rescue:Resonator-Device-Принципиально-rescue ZQ1
 U 1 1 61684E3A
 P 12900 3550
@@
 	12350 3550 12350 2550
 $Comp
-L power:Earth #PWR?
+L Prinsip-rescue:Earth-power #PWR?
 U 1 1 616A9422
 P 12900 3750
@@
 $EndComp
 $Comp
-L Принципиально-rescue:R_Small-Device R2
+L Prinsip-rescue:R_Small-Device-Принципиально-rescue R2
 U 1 1 616AA0CB
 P 13450 3050
@@
 $EndComp
 $Comp
-L Принципиально-rescue:R_Small-Device R1
+L Prinsip-rescue:R_Small-Device-Принципиально-rescue R1
 U 1 1 616AAF02
 P 12900 1800
@@
 CLK
 $Comp
-L Принципиально-rescue:TAB-Prinsip U?
+L Prinsip-rescue:TAB-Prinsip-Принципиально-rescue U?
 U 1 1 61723B06
 P 13950 8150
@@
 	1    0    0    -1
 $EndComp
+$Comp
+L rescue:con-Prinsip C1
+U 1 1 616915C1
+P 15150 8200
+F 0 "C1" H 15125 8283 50  0000 C CNN
+F 1 "con-Prinsip" H 15125 8284 50  0001 C CNN
+F 2 "" H 15200 8500 50  0001 C CNN
+F 3 "" H 15200 8500 50  0001 C CNN
+	1    15150 8200
+	1    0    0    -1
+$EndComp
+$Comp
+L rescue:con-Prinsip C2...C4
+U 1 1 6169254A
+P 15150 8600
+F 0 "C2...C4" H 15125 8683 50  0000 C CNN
+F 1 "con-Prinsip" H 15125 8684 50  0001 C CNN
+F 2 "" H 15200 8900 50  0001 C CNN
+F 3 "" H 15200 8900 50  0001 C CNN
+	1    15150 8600
+	1    0    0    -1
+$EndComp
+Wire Wire Line
+	14850 8000 15000 8000
+Wire Wire Line
+	15000 8000 15000 8250
+Connection ~ 15000 8250
+Wire Wire Line
+	15000 8250 15000 8650
+Wire Wire Line
+	14850 7850 15250 7850
+Wire Wire Line
+	15250 7850 15250 8250
+Connection ~ 15250 8250
+Wire Wire Line
+	15250 8250 15250 8650
+Text Notes 15150 8250 0    79   ~ 0
++
 $EndSCHEMATC

Commit message: added fio
Connections:
- new net: DD40.~ (~LD), DD41.~ (Uоп) (x8)
- new net: C1.~, C2...C4.~
Changed lines of the file:
@@
 Comp "МГТУ им. Н.Э. Баумана\\nгруппа ИУ6-64Б"
 Comment1 "Генератор пилы на ЦАП"
-Comment2 ""
+Comment2 "Прохорова А.В."
 Comment3 "Захаров М.А."
 Comment4 ""
@@
 	1    0    0    -1
 $EndComp
-Wire Wire Line
-	14850 8000 15000 8000
-Wire Wire Line
-	15000 8000 15000 8250
-Connection ~ 15000 8250
-Wire Wire Line
-	15000 8250 15000 8650
-Wire Wire Line
-	14850 7850 15250 7850
-Wire Wire Line
-	15250 7850 15250 8250
-Connection ~ 15250 8250
-Wire Wire Line
-	15250 8250 15250 8650
 Text Notes 15150 8250 0    79   ~ 0
 +
+Wire Wire Line
+	14850 8000 14900 8000
+Wire Wire Line
+	14900 8000 14900 8250
+Wire Wire Line
+	14900 8650 15000 8650
+Wire Wire Line
+	15250 8650 15350 8650
+Wire Wire Line
+	15350 8650 15350 8250
+Wire Wire Line
+	14850 7850 15350 7850
+Wire Wire Line
+	15250 8250 15350 8250
+Connection ~ 15350 8250
+Wire Wire Line
+	15350 8250 15350 7850
+Wire Wire Line
+	15000 8250 14900 8250
+Connection ~ 14900 8250
+Wire Wire Line
+	14900 8250 14900 8650
 $EndSCHEMATC

Commit message: Updated pdf
Connections:
- new net: DD40.~ (~LD), DD41.~ (Uоп) (x8)
- new net: C1.~, C2...C4.~
Other:
- note added: "Контакт 16 микросхем\nDD39, DD40, DD41\nподключить к VCC"
- note added: "Контакт 8 микросхем\nDD39, DD40, DD41\nподключить к GND"
- moved on the sheet: C1, C2...C4
Changed lines of the file:
@@
 L Prinsip-rescue:TAB-Prinsip-Принципиально-rescue U?
 U 1 1 61723B06
-P 13950 8150
-F 0 "U?" H 14878 8474 50  0001 L CNN
-F 1 "TAB-Prinsip" H 14878 8429 50  0001 L CNN
-F 2 "" H 12600 9250 50  0001 C CNN
-F 3 "" H 12600 9250 50  0001 C CNN
-	1    13950 8150
+P 12450 7700
+F 0 "U?" H 13378 8024 50  0001 L CNN
+F 1 "TAB-Prinsip" H 13378 7979 50  0001 L CNN
+F 2 "" H 11100 8800 50  0001 C CNN
+F 3 "" H 11100 8800 50  0001 C CNN
+	1    12450 7700
 	1    0    0    -1
 $EndComp
@@
 L rescue:con-Prinsip C1
 U 1 1 616915C1
-P 15150 8200
-F 0 "C1" H 15125 8283 50  0000 C CNN
-F 1 "con-Prinsip" H 15125 8284 50  0001 C CNN
-F 2 "" H 15200 8500 50  0001 C CNN
-F 3 "" H 15200 8500 50  0001 C CNN
-	1    15150 8200
+P 13650 7750
+F 0 "C1" H 13625 7833 50  0000 C CNN
+F 1 "con-Prinsip" H 13625 7834 50  0001 C CNN
+F 2 "" H 13700 8050 50  0001 C CNN
+F 3 "" H 13700 8050 50  0001 C CNN
+	1    13650 7750
 	1    0    0    -1
 $EndComp
@@
 L rescue:con-Prinsip C2...C4
 U 1 1 6169254A
-P 15150 8600
-F 0 "C2...C4" H 15125 8683 50  0000 C CNN
-F 1 "con-Prinsip" H 15125 8684 50  0001 C CNN
-F 2 "" H 15200 8900 50  0001 C CNN
-F 3 "" H 15200 8900 50  0001 C CNN
-	1    15150 8600
+P 13650 8150
+F 0 "C2...C4" H 13625 8233 50  0000 C CNN
+F 1 "con-Prinsip" H 13625 8234 50  0001 C CNN
+F 2 "" H 13700 8450 50  0001 C CNN
+F 3 "" H 13700 8450 50  0001 C CNN
+	1    13650 8150
 	1    0    0    -1
 $EndComp
-Text Notes 15150 8250 0    79   ~ 0
+Text Notes 13650 7800 0    79   ~ 0
 +
 Wire Wire Line
-	14850 8000 14900 8000
+	13350 7550 13400 7550
 Wire Wire Line
-	14900 8000 14900 8250
+	13400 7550 13400 7800
 Wire Wire Line
-	14900 8650 15000 8650
+	13400 8200 13500 8200
 Wire Wire Line
-	15250 8650 15350 8650
+	13750 8200 13850 8200
 Wire Wire Line
-	15350 8650 15350 8250
+	13850 8200 13850 7800
 Wire Wire Line
-	14850 7850 15350 7850
+	13350 7400 13850 7400
 Wire Wire Line
-	15250 8250 15350 8250
-Connection ~ 15350 8250
+	13750 7800 13850 7800
+Connection ~ 13850 7800
 Wire Wire Line
-	15350 8250 15350 7850
+	13850 7800 13850 7400
 Wire Wire Line
-	15000 8250 14900 8250
-Connection ~ 14900 8250
+	13500 7800 13400 7800
+Connection ~ 13400 7800
 Wire Wire Line
-	14900 8250 14900 8650
+	13400 7800 13400 8200
+Text Notes 14300 7250 0    79   ~ 0
+Контакт 16 микросхем\nDD39, DD40, DD41\nподключить к VCC
+Text Notes 14300 7950 0    79   ~ 0
+Контакт 8 микросхем\nDD39, DD40, DD41\nподключить к GND
 $EndSCHEMATC
