File: Func/Func/Func.sch (KiCad schematic (older format))
At the start: 6 parts

Commit message: Updated
Parts:
- added U?: KEY, symbol Func:KEY
Connections:
- wire segments 17 -> 21
Changed lines of the file:
@@
 L Func:CLK U?
 U 1 1 6167F422
-P 4650 6650
-F 0 "U?" H 4708 6765 50  0001 C CNN
-F 1 "CLK" H 4708 6674 50  0001 C CNN
-F 2 "" H 4650 6650 50  0001 C CNN
-F 3 "" H 4650 6650 50  0001 C CNN
-	1    4650 6650
+P 4550 7200
+F 0 "U?" H 4608 7315 50  0001 C CNN
+F 1 "CLK" H 4608 7224 50  0001 C CNN
+F 2 "" H 4550 7200 50  0001 C CNN
+F 3 "" H 4550 7200 50  0001 C CNN
+	1    4550 7200
 	1    0    0    -1
 $EndComp
@@
 L Func:CMP U?
 U 1 1 6167F9AA
-P 5150 5150
-F 0 "U?" H 5158 5265 50  0001 C CNN
-F 1 "CMP" H 5158 5174 50  0001 C CNN
-F 2 "" H 5150 5150 50  0001 C CNN
-F 3 "" H 5150 5150 50  0001 C CNN
-	1    5150 5150
+P 5150 4900
+F 0 "U?" H 5158 5015 50  0001 C CNN
+F 1 "CMP" H 5158 4924 50  0001 C CNN
+F 2 "" H 5150 4900 50  0001 C CNN
+F 3 "" H 5150 4900 50  0001 C CNN
+	1    5150 4900
 	1    0    0    -1
 $EndComp
@@
 +21V
 Wire Wire Line
-	10750 5800 11000 5800
-Wire Wire Line
-	5600 7150 6200 7150
-Wire Wire Line
 	6200 7150 6200 6100
 Wire Wire Line
@@
 Wire Wire Line
 	8150 7150 6200 7150
-Connection ~ 6200 7150
 Wire Wire Line
 	8100 5850 8100 5750
@@
 8
 Wire Wire Line
-	6050 5600 6500 5600
-Wire Wire Line
 	7750 5850 7750 4300
 Wire Wire Line
 	7750 4300 4050 4300
 Wire Wire Line
-	4050 4300 4050 5600
+	4050 4300 4050 5350
 Wire Wire Line
-	4050 5600 4400 5600
+	4050 5350 4400 5350
 Wire Wire Line
 	7450 5850 7750 5850
@@
 Wire Wire Line
 	7750 5850 8100 5850
-Entry Wire Line
-	4350 5550 4450 5650
-Text Notes 4300 5500 0    50   ~ 0
+Text Notes 4300 5250 0    50   ~ 0
 8
 Wire Wire Line
@@
 Entry Wire Line
 	9150 5700 9250 5800
+Entry Wire Line
+	4350 5300 4450 5400
+$Comp
+L Func:KEY U?
+U 1 1 6168002D
+P 2750 5900
+F 0 "U?" H 3078 5646 50  0001 L CNN
+F 1 "KEY" H 3078 5600 50  0001 L CNN
+F 2 "" H 2750 5900 50  0001 C CNN
+F 3 "" H 2750 5900 50  0001 C CNN
+	1    2750 5900
+	1    0    0    -1
+$EndComp
+Wire Wire Line
+	3000 6200 4400 6200
+Entry Wire Line
+	4350 6150 4450 6250
+Wire Wire Line
+	5500 7700 6200 7700
+Wire Wire Line
+	6200 7700 6200 7150
+Connection ~ 6200 7150
+Wire Wire Line
+	6050 5350 6300 5350
+Wire Wire Line
+	6300 5350 6300 5600
+Wire Wire Line
+	6300 5600 6500 5600
+Wire Wire Line
+	10750 5800 10900 5800
 $EndSCHEMATC
