File: Func/Func/Func.sch (KiCad schematic (older format))
At the start: 7 parts

Commit message: Updated
Other:
- note added: "1"
- note added: "2"
- note added: "3"
- note added: "4"
- note added: "5"
- note added: "6"
- note added: "7"
Changed lines of the file:
@@
 L Func:CLK U?
 U 1 1 6167F422
-P 4550 7200
-F 0 "U?" H 4608 7315 50  0001 C CNN
-F 1 "CLK" H 4608 7224 50  0001 C CNN
-F 2 "" H 4550 7200 50  0001 C CNN
-F 3 "" H 4550 7200 50  0001 C CNN
-	1    4550 7200
+P 5150 7200
+F 0 "U?" H 5208 7315 50  0001 C CNN
+F 1 "CLK" H 5208 7224 50  0001 C CNN
+F 2 "" H 5150 7200 50  0001 C CNN
+F 3 "" H 5150 7200 50  0001 C CNN
+	1    5150 7200
 	1    0    0    -1
 $EndComp
@@
 L Func:RECV U?
 U 1 1 61681546
-P 11500 5600
-F 0 "U?" H 11828 5446 50  0001 L CNN
-F 1 "RECV" H 11828 5355 50  0001 L CNN
-F 2 "" H 11500 5600 50  0001 C CNN
-F 3 "" H 11500 5600 50  0001 C CNN
-	1    11500 5600
+P 11500 5500
+F 0 "U?" H 11828 5346 50  0001 L CNN
+F 1 "RECV" H 11828 5255 50  0001 L CNN
+F 2 "" H 11500 5500 50  0001 C CNN
+F 3 "" H 11500 5500 50  0001 C CNN
+	1    11500 5500
 	1    0    0    -1
 $EndComp
@@
 	4350 6150 4450 6250
 Wire Wire Line
-	5500 7700 6200 7700
+	6100 7700 6200 7700
 Wire Wire Line
 	6200 7700 6200 7150
@@
 Wire Wire Line
 	6300 5600 6500 5600
-Wire Wire Line
-	10750 5800 10900 5800
 Entry Wire Line
 	2950 6150 3050 6250
 Text Notes 3000 6200 0    50   ~ 0
 8
-Text Notes 4250 6150 0    50   ~ 0
+Text Notes 4300 6150 0    50   ~ 0
 8
+Text Notes 5050 6500 0    118  ~ 0
+2
+Text Notes 5050 8100 0    118  ~ 0
+3
+Text Notes 7000 6150 0    118  ~ 0
+4
+Text Notes 8850 6150 0    118  ~ 0
+5
+Text Notes 10250 6050 0    118  ~ 0
+6
+Wire Wire Line
+	10750 5800 10900 5800
+Text Notes 11450 6050 0    118  ~ 0
+7
+Text Notes 2700 6400 0    118  ~ 0
+1
 $EndSCHEMATC
